File: hardware/adapter_chronos_helios/chronos_helios_adapter.kicad_pcb (KiCad board)
At the start: 4 copper layers, 28 x 28 mm, 11 parts, among them J1 FPC-05F-22PH20, J2 F0502-B-15-15T-R

Commit message: hardware: adapter v3 - user-verified pin-1 sides, Helios link maps straight
Physical check on the boards showed both pin 1s on the same absolute side (Helios CAM connector is opposite-handed vs standard FH12), so the 15p link maps straight (CAM.j <-> J2.j) instead of mirrored. All six CSI conductors now route as identical top-layer diagonals with zero vias; only the SDA/SCL swap crosses on In2.Cu. Added _check_map.py end-to-end signal-map verification (PASS). DRC 0 errors.

Co-authored-by: Cursor <cursoragent@cursor.com>
Parts:
- moved TP2 11.4 mm to (106.2, 107.8)
- moved TP3 11.4 mm to (117.6, 107.8)
Connections:
- J2 pad 1: V33_HELIOS -> SENSE_H
- J2 pad 10: CSI_D1_P -> GND
- J2 pad 11: CSI_D1_N -> (no net)
- J2 pad 12: GND -> (no net)
- J2 pad 13: CSI_D0_P -> I2C_SCL
- J2 pad 14: CSI_D0_N -> I2C_SDA
- J2 pad 15: SENSE_H -> V33_HELIOS
- J2 pad 2: I2C_SDA -> CSI_D0_N
- J2 pad 3: I2C_SCL -> CSI_D0_P
- J2 pad 4: (no net) -> GND
- J2 pad 5: (no net) -> CSI_D1_N
- J2 pad 6: GND -> CSI_D1_P
- J2 pad 7: CSI_CLK_P -> GND
- J2 pad 9: GND -> CSI_CLK_P
Routing:
- net I2C_SCL: track 24.4 -> 9.41 mm, vias 2 -> 0
- net V33_HELIOS: track 19.2 -> 6.60 mm, vias 2 -> 0
- net I2C_SDA: track 19.9 -> 9.72 mm
- net CSI_D0_N: track 17.7 -> 9.51 mm, vias 2 -> 0
- net CSI_D0_P: track 16.1 -> 9.51 mm, vias 2 -> 0
- net CSI_D1_N: track 14.7 -> 9.51 mm, vias 2 -> 0
- net CSI_D1_P: track 13.1 -> 9.51 mm, vias 2 -> 0
- net CSI_CLK_N: track 12.2 -> 9.51 mm, vias 2 -> 0
- net CSI_CLK_P: track 10.1 -> 9.51 mm, vias 2 -> 0
Other:
- board text added: "CHRONOS-HELIOS ADAPTER v3"
- board text added: "STRAIGHT MAP + I2C SWAP ON BOARD"
- board text removed: "CHRONOS-HELIOS ADAPTER v2"
- board text removed: "CROSSOVER ON BOARD"
